Commit message: working on the wheel mesh.

File: jetduinobot_description/urdf/jetduinobot.urdf (robot description, URDF)
Before this commit: robot None, 6 links, 5 joints
Links:
- link left_front_wheel_link: geometry collision cylinder length=0.025 radius=0.029; visual mesh filename=package://jetduinobot_description/meshes/wheel_tread.dae scale=1 1 1
- link left_rear_wheel_link: geometry collision cylinder length=0.025 radius=0.029; visual mesh filename=package://jetduinobot_description/meshes/wheel_tread.dae
- link right_front_wheel_link: geometry collision cylinder length=0.025 radius=0.029; visual mesh filename=package://jetduinobot_description/meshes/wheel_tread.dae
- link right_rear_wheel_link: geometry collision cylinder length=0.025 radius=0.029; visual mesh filename=package://jetduinobot_description/meshes/wheel_tread.dae scale=3 3 3
Joints:
- joint right_rear_wheel_joint: origin xyz=-0.0825 -0.074 -0.062 rpy=-1.5708 0 0 -> xyz=-1.0825 -0.074 -0.062 rpy=-1.5708 0 0

Commit message: Got the chassis loading in ros, but the wheel is not showing any materials.

File: jetduinobot_description/urdf/jetduinobot.urdf (robot description, URDF)
Before this commit: robot jetduinobot, 6 links, 5 joints
Links:
- link base_link: geometry collision box size=0.185 0.23 0.058; visual mesh filename=package://jetduinobot_description/meshes/chassis.dae scale=0.1 0.1 0.1
- link left_front_wheel_link: geometry collision cylinder length=0.025 radius=0.029; visual mesh filename=package://jetduinobot_description/meshes/wheel.dae scale=0.1 0.1 0.1
- link left_rear_wheel_link: geometry collision cylinder length=0.025 radius=0.029; visual mesh filename=package://jetduinobot_description/meshes/wheel.dae scale=0.1 0.1 0.1
- link right_front_wheel_link: geometry collision cylinder length=0.025 radius=0.029; visual mesh filename=package://jetduinobot_description/meshes/wheel.dae scale=0.1 0.1 0.1
- link right_rear_wheel_link: geometry collision cylinder length=0.025 radius=0.029; visual mesh filename=package://jetduinobot_description/meshes/wheel.dae scale=0.1 0.1 0.1

Commit message: I got the base urdf file setup and working. Now I need to get the xacro version working. Still need to add jetson and other parts and get masses and inertias setup correctly.

File: jetduinobot_description/urdf/jetduinobot.urdf (robot description, URDF)
Before this commit: robot jetduinobot, 6 links, 5 joints
Links:
- link base_link: geometry collision box size=0.185 0.225 0.058; visual mesh filename=package://jetduinobot_description/meshes/chassis.dae scale=0.1 0.1 0.1
Joints:
- joint left_front_wheel_joint: origin xyz=0.0475 0.074 -0.062 rpy=-1.5708 0 0 -> xyz=0.07 0.0455 -0.017 rpy=0 1.5708 0
- joint left_rear_wheel_joint: origin xyz=-0.0825 0.074 -0.062 rpy=-1.5708 0 0 -> xyz=0.07 -0.0875 -0.017 rpy=0 1.5708 0
- joint right_front_wheel_joint: origin xyz=0.0475 -0.074 -0.062 rpy=-1.5708 0 0 -> xyz=-0.07 0.0455 -0.017 rpy=0 -1.5708 0
- joint right_rear_wheel_joint: origin xyz=-1.0825 -0.074 -0.062 rpy=-1.5708 0 0 -> xyz=-0.07 -0.0875 -0.017 rpy=0 -1.5708 0

Commit message: renmaed the images to use lower case extension. Added tk1 to urdf for testing.

File: jetduinobot_description/urdf/jetduinobot.urdf (robot description, URDF)
Before this commit: robot jetduinobot, 6 links, 5 joints
Links:
- added link jetson_tk1_link, mass 0.5; collision box size=0.185 0.225 0.058; visual mesh filename=package://jetduinobot_description/meshes/jetson_tk1/jetson_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 scale=0.1 0.1 0.1
- link left_front_wheel_link: geometry collision cylinder length=0.025 radius=0.029; visual mesh filename=package://jetduinobot_description/meshes/wheel/wheel.dae scale=0.1 0.1 0.1
- link left_rear_wheel_link: geometry collision cylinder length=0.025 radius=0.029; visual mesh filename=package://jetduinobot_description/meshes/wheel/wheel.dae scale=0.1 0.1 0.1
- link right_front_wheel_link: geometry collision cylinder length=0.025 radius=0.029; visual mesh filename=package://jetduinobot_description/meshes/wheel/wheel.dae scale=0.1 0.1 0.1
- link right_rear_wheel_link: geometry collision cylinder length=0.025 radius=0.029; visual mesh filename=package://jetduinobot_description/meshes/wheel/wheel.dae scale=0.1 0.1 0.1
Joints:
- added joint jetson_tk1_joint: type fixed, parent base_link, child jetson_tk1_link, origin xyz=0 0 1 rpy=0 0 0
