Commit message: renamed the jetduinoBot urdf to be a test version.

File: jetduinobot_description/urdf/jetduinobot_test.urdf (robot description, URDF)
Before this commit: robot jetduinobot, 7 links, 6 joints
Links:
- link jetson_tk1_link: geometry collision box size=0.185 0.225 0.058; visual mesh filename=package://jetduinobot_description/meshes/top_plate.dae scale=0.1 0.1 0.1
