Commit message: Trying to get the urdf to work. It is not wanting to load the dae files.

File: jetduinobot_description/urdf/dfrobot_4wd.urdf.xacro (robot description, xacro)
@@ -1,4 +1,4 @@
 <?xml version="1.0"?>
-<robot name="jetduino_bot" xmlns:xacro="http://ros.org/wiki/xacro">
+<robot xmlns:xacro="http://ros.org/wiki/xacro">
   <link name="world_link" />
   <link name="base_link">
@@ -7,7 +7,5 @@
         <box size="0.225 0.185 0.15"/>
       </geometry>
-      <material name="silver">
-        <color rgba="0.75 0.75 0.75 1"/>
-      </material>
+      <material name="silver" />
     </visual>
     <collision>
@@ -31,13 +29,10 @@
     <visual>
       <geometry>
-        <cylinder length="0.025" radius="0.0325"/>
+        <mesh filename="$(find jetduinobot_description)/meshes/wheel.dae"/>
       </geometry>
-      <material name="black">
-        <color rgba="0 0 0 1"/>
-      </material>
     </visual>
     <collision>
       <geometry>
-        <cylinder length="0.025" radius="0.0325"/>
+        <cylinder length="0.025" radius="0.029"/>
       </geometry>
     </collision>
@@ -57,5 +52,5 @@
     <visual>
       <geometry>
-        <cylinder length="0.025" radius="0.0325"/>
+        <mesh filename="$(find jetduinobot_description)/meshes/wheel.dae"/>
       </geometry>
       <material name="black"/>
@@ -63,5 +58,5 @@
     <collision>
       <geometry>
-        <cylinder length="0.025" radius="0.0325"/>
+        <cylinder length="0.025" radius="0.029"/>
       </geometry>
     </collision>
@@ -82,5 +77,5 @@
     <visual>
       <geometry>
-        <cylinder length="0.025" radius="0.0325"/>
+        <mesh filename="$(find jetduinobot_description)/meshes/wheel.dae"/>
       </geometry>
       <material name="black"/>
@@ -88,5 +83,5 @@
     <collision>
       <geometry>
-        <cylinder length="0.025" radius="0.0325"/>
+        <cylinder length="0.025" radius="0.029"/>
       </geometry>
     </collision>
@@ -106,5 +101,5 @@
     <visual>
       <geometry>
-        <cylinder length="0.025" radius="0.0325"/>
+        <mesh filename="$(find jetduinobot_description)/meshes/wheel.dae"/>
       </geometry>
       <material name="black"/>
@@ -112,5 +107,5 @@
     <collision>
       <geometry>
-        <cylinder length="0.025" radius="0.0325"/>
+        <cylinder length="0.025" radius="0.029"/>
       </geometry>
     </collision>

File: jetduinobot_description/urdf/jetduinobot.urdf.xacro (robot description, xacro)
@@ -3,5 +3,5 @@
   The complete jetduinobot library of xacros for easy reference
  -->
-<robot xmlns:xacro="http://ros.org/wiki/xacro">
+<robot xmlns:xacro="http://ros.org/wiki/xacro" name="jetduinobot">
   <!-- General -->
   <xacro:include filename="$(find jetduinobot_description)/urdf/common_properties.urdf.xacro"/>

File: jetduinobot_description/urdf/jetduinobot_properties.urdf.xacro (robot description, xacro)
@@ -7,4 +7,3 @@
     http://www.ros.org/reps/rep-0119.html
    -->
-  <!--
 </robot>

Commit message: 1. added masses file. 2. started modifying the xacro file for the chassis 3. tweaked the chassis collada file to get the grove_motor textures.

File: jetduinobot_description/urdf/dfrobot_4wd.urdf.xacro (robot description, xacro)
@@ -1,20 +1,27 @@
 <?xml version="1.0"?>
 <robot xmlns:xacro="http://ros.org/wiki/xacro">
+  <xacro:property name="chassis_length" value="0.225" />
+  <xacro:property name="chassis_width" value="0.185" />
+  <xacro:property name="chassis_height" value="0.058" />
+  <xacro:property name="chassis_mass" value="0.416" />
   <link name="world_link" />
   <link name="base_link">
     <visual>
       <geometry>
-        <box size="0.225 0.185 0.15"/>
+        <mesh filename="package://jetduinobot_description/meshes/chassis.dae" scale="0.1 0.1 0.1"/>
       </geometry>
+      <origin rpy="0 0 0" xyz="0 -0.0075 -0.029"/>
       <material name="silver" />
     </visual>
     <collision>
       <geometry>
-        <box size="0.225 0.185 0.15"/>
+        <box size="${chassis_width} ${chassis_length} ${chassis_height}"/>
       </geometry>
     </collision>
     <inertial>
-      <mass value="0.5"/>
-      <inertia ixx="0.015" iyy="0.0375" izz="0.0375" ixy="0" ixz="0" iyz="0"/>
+      <mass value="${chassis_mass}"/>
+      <inertia ixx="${0.0833 * chassis_mass * (chassis_height*chassis_height + chassis_length*chassis_length)}" ixy="0" ixz="0"
+               iyy="${0.0833 * chassis_mass * (chassis_width*chassis_width + chassis_length*chassis_length)}" iyz="0"
+               izz="${0.0833 * chassis_mass * (chassis_height*chassis_height + chassis_width*chassis_width)}" />
     </inertial>
   </link>
@@ -24,4 +31,7 @@
     <origin rpy="0 0 0" xyz="0 0 0"/>
   </joint>
+  <xacro:property name="wheel_length" value="0.025" />
+  <xacro:property name="chassis_radius" value="0.029" />
+  <xacro:property name="wheel_mass" value="0.030" />
   <!-- rear wheels -->
   <!-- right rear wheel -->
@@ -29,15 +39,17 @@
     <visual>
       <geometry>
-        <mesh filename="$(find jetduinobot_description)/meshes/wheel_tread.dae"/>
+        <mesh filename="package://jetduinobot_description/meshes/wheel/wheel.dae" scale="0.1 0.1 0.1"/>
       </geometry>
     </visual>
     <collision>
       <geometry>
-        <cylinder length="0.025" radius="0.029"/>
+        <cylinder length="${wheel_length}" radius="${wheel_radius}"/>
       </geometry>
     </collision>
     <inertial>
-      <mass value="0.05"/>
-      <inertia ixx="5.1458e-5" iyy="5.1458e-5" izz="6.125e-5" ixy="0" ixz="0" iyz="0"/>
+      <mass value="${wheel_mass}"/>
+      <inertia ixx="${0.0833 * wheel_mass * (3*wheel_radius*wheel_radius + wheel_length*wheel_length)}" ixy="0" ixz="0"
+               iyy="${0.0833 * wheel_mass * (3*wheel_radius*wheel_radius + wheel_length*wheel_length)}" iyz="0"
+               izz="${0.0833 * wheel_mass * (3*wheel_radius*wheel_radius + wheel_length*wheel_length)}" />
     </inertial>
   </link>
@@ -46,5 +58,5 @@
     <parent link="base_link"/>
     <child link="right_rear_wheel_link"/>
-    <origin rpy="-1.5708 0 0" xyz="-0.0825 -0.074 -0.062"/>
+    <origin rpy="0 -1.5708 0" xyz="-0.07 -0.0875 -0.017"/>
   </joint>
   <!-- left rear wheel -->
@@ -52,16 +64,17 @@
     <visual>
       <geometry>
-        <mesh filename="$(find jetduinobot_description)/meshes/wheel_tread.dae"/>
+        <mesh filename="package://jetduinobot_description/meshes/wheel/wheel.dae" scale="0.1 0.1 0.1"/>
       </geometry>
-      <material name="black"/>
     </visual>
     <collision>
       <geometry>
-        <cylinder length="0.025" radius="0.029"/>
+        <cylinder length="${wheel_length}" radius="${wheel_radius}"/>
       </geometry>
     </collision>
     <inertial>
-      <mass value="0.1"/>
-      <inertia ixx="5.1458e-5" iyy="5.1458e-5" izz="6.125e-5" ixy="0" ixz="0" iyz="0"/>
+      <mass value="${wheel_mass}"/>
+      <inertia ixx="${0.0833 * wheel_mass * (3*wheel_radius*wheel_radius + wheel_length*wheel_length)}" ixy="0" ixz="0"
+               iyy="${0.0833 * wheel_mass * (3*wheel_radius*wheel_radius + wheel_length*wheel_length)}" iyz="0"
+               izz="${0.0833 * wheel_mass * (3*wheel_radius*wheel_radius + wheel_length*wheel_length)}" />
     </inertial>
   </link>
@@ -70,5 +83,5 @@
     <parent link="base_link"/>
     <child link="left_rear_wheel_link"/>
-    <origin rpy="-1.5708 0 0" xyz="-0.0825 0.074 -0.062"/>
+    <origin rpy="0 1.5708 0" xyz="0.07 -0.0875 -0.017"/>
   </joint>
   <!-- front wheels -->
@@ -77,16 +90,17 @@
     <visual>
       <geometry>
-        <mesh filename="$(find jetduinobot_description)/meshes/wheel_tread.dae"/>
+        <mesh filename="package://jetduinobot_description/meshes/wheel/wheel.dae" scale="0.1 0.1 0.1"/>
       </geometry>
-      <material name="black"/>
     </visual>
     <collision>
       <geometry>
-        <cylinder length="0.025" radius="0.029"/>
+        <cylinder length="${wheel_length}" radius="${wheel_radius}"/>
       </geometry>
     </collision>
     <inertial>
-      <mass value="0.05"/>
-      <inertia ixx="5.1458e-5" iyy="5.1458e-5" izz="6.125e-5" ixy="0" ixz="0" iyz="0"/>
+      <mass value="${wheel_mass}"/>
+      <inertia ixx="${0.0833 * wheel_mass * (3*wheel_radius*wheel_radius + wheel_length*wheel_length)}" ixy="0" ixz="0"
+               iyy="${0.0833 * wheel_mass * (3*wheel_radius*wheel_radius + wheel_length*wheel_length)}" iyz="0"
+               izz="${0.0833 * wheel_mass * (3*wheel_radius*wheel_radius + wheel_length*wheel_length)}" />
     </inertial>
   </link>
@@ -95,5 +109,5 @@
     <parent link="base_link"/>
     <child link="right_front_wheel_link"/>
-    <origin rpy="-1.5708 0 0" xyz="0.0475 -0.074 -0.062"/>
+    <origin rpy="0 -1.5708 0" xyz="-0.07 0.0455 -0.017"/>
   </joint>
   <!-- left front wheel -->
@@ -101,16 +115,17 @@
     <visual>
       <geometry>
-        <mesh filename="$(find jetduinobot_description)/meshes/wheel_tread.dae"/>
+        <mesh filename="package://jetduinobot_description/meshes/wheel/wheel.dae" scale="0.1 0.1 0.1"/>
       </geometry>
-      <material name="black"/>
     </visual>
     <collision>
       <geometry>
-        <cylinder length="0.025" radius="0.029"/>
+        <cylinder length="${wheel_length}" radius="${wheel_radius}"/>
       </geometry>
     </collision>
     <inertial>
-      <mass value="0.1"/>
-      <inertia ixx="5.1458e-5" iyy="5.1458e-5" izz="6.125e-5" ixy="0" ixz="0" iyz="0"/>
+      <mass value="${wheel_mass}"/>
+      <inertia ixx="${0.0833 * wheel_mass * (3*wheel_radius*wheel_radius + wheel_length*wheel_length)}" ixy="0" ixz="0"
+               iyy="${0.0833 * wheel_mass * (3*wheel_radius*wheel_radius + wheel_length*wheel_length)}" iyz="0"
+               izz="${0.0833 * wheel_mass * (3*wheel_radius*wheel_radius + wheel_length*wheel_length)}" />
     </inertial>
   </link>
@@ -119,5 +134,5 @@
     <parent link="base_link"/>
     <child link="left_front_wheel_link"/>
-    <origin rpy="-1.5708 0 0" xyz="0.0475 0.074 -0.062"/>
+    <origin rpy="0 1.5708 0" xyz="0.07 0.0455 -0.017"/>
   </joint>
   <gazebo>

Commit message: added the battery to the base xacro file.

File: jetduinobot_description/urdf/dfrobot_4wd.urdf.xacro (robot description, xacro)
@@ -31,6 +31,36 @@
     <origin rpy="0 0 0" xyz="0 0 0"/>
   </joint>
+  <!-- battery -->
+  <xacro:property name="battery_length" value="0.13" />
+  <xacro:property name="battery_width" value="0.045" />
+  <xacro:property name="battery_height" value="0.0025" />
+  <xacro:property name="battery_mass" value="0.330" />
+  <link name="battery_link">
+    <visual>
+      <geometry>
+        <mesh filename="package://jetduinobot_description/meshes/battery_large/battery_large.dae"/>
+      </geometry>
+      <material name="black" />
+    </visual>
+    <collision>
+      <geometry>
+        <box size="${battery_width} ${battery_length} ${battery_height}"/>
+      </geometry>
+    </collision>
+    <inertial>
+      <mass value="${battery_mass}"/>
+      <inertia ixx="${0.0833 * battery_mass * (battery_height*battery_height + battery_length*battery_length)}" ixy="0" ixz="0"
+               iyy="${0.0833 * battery_mass * (battery_width*battery_width + battery_length*battery_length)}" iyz="0"
+               izz="${0.0833 * battery_mass * (battery_height*battery_height + battery_width*battery_width)}" />
+    </inertial>
+  </link>
+  <joint name="batteryjoint" type="fixed">
+    <parent link="base_link"/>
+    <child link="battery_link"/>
+    <origin rpy="0 0 1.5708" xyz="0 -0.02 0.015"/>
+  </joint>
+  <!-- wheels -->
   <xacro:property name="wheel_length" value="0.025" />
-  <xacro:property name="chassis_radius" value="0.029" />
+  <xacro:property name="wheel_radius" value="0.029" />
   <xacro:property name="wheel_mass" value="0.030" />
   <!-- rear wheels -->
@@ -41,4 +71,5 @@
         <mesh filename="package://jetduinobot_description/meshes/wheel/wheel.dae" scale="0.1 0.1 0.1"/>
       </geometry>
+      <material name="black" />
     </visual>
     <collision>
@@ -66,4 +97,5 @@
         <mesh filename="package://jetduinobot_description/meshes/wheel/wheel.dae" scale="0.1 0.1 0.1"/>
       </geometry>
+      <material name="black" />
     </visual>
     <collision>
@@ -92,4 +124,5 @@
         <mesh filename="package://jetduinobot_description/meshes/wheel/wheel.dae" scale="0.1 0.1 0.1"/>
       </geometry>
+      <material name="black" />
     </visual>
     <collision>
@@ -117,4 +150,5 @@
         <mesh filename="package://jetduinobot_description/meshes/wheel/wheel.dae" scale="0.1 0.1 0.1"/>
       </geometry>
+      <material name="black" />
     </visual>
     <collision>

Commit message: Got the jetduino on the model, but I think I want to modify it to spread the dc-converter out to reduce height.

File: jetduinobot_description/urdf/dfrobot_4wd.urdf.xacro (robot description, xacro)
@@ -64,4 +64,5 @@
   <xacro:property name="wheel_radius" value="0.029" />
   <xacro:property name="wheel_mass" value="0.030" />
+  <xacro:property name="wheel_separation" value="0.148" />
   <!-- rear wheels -->
   <!-- right rear wheel -->
@@ -176,6 +177,6 @@
       <leftRearJoint>left_rear_wheel_joint</leftRearJoint>
       <rightRearJoint>right_rear_wheel_joint</rightRearJoint>
-      <wheelSeparation>0.148</wheelSeparation>
-      <wheelDiameter>0.065</wheelDiameter>
+      <wheelSeparation>${wheel_separation}</wheelSeparation>
+      <wheelDiameter>${2 * wheel_radius}</wheelDiameter>
       <robotBaseFrame>base_link</robotBaseFrame>
       <torque>20</torque>

File: jetduinobot_description/urdf/jetduinobot.urdf.xacro (robot description, xacro)
@@ -9,4 +9,5 @@
   <!-- Bases -->
   <xacro:include filename="$(find jetduinobot_description)/urdf/dfrobot_4wd.urdf.xacro"/>
+  <xacro:include filename="$(find jetduinobot_description)/urdf/jetduino.urdf.xacro"/>
   <!-- Stacks -->
   <!-- 3D Sensors -->

Commit message: tweaked the materials in the xacro file.

File: jetduinobot_description/urdf/dfrobot_4wd.urdf.xacro (robot description, xacro)
@@ -12,5 +12,5 @@
       </geometry>
       <origin rpy="0 0 0" xyz="0 -0.0075 -0.029"/>
-      <material name="silver" />
+      <xacro:insert_block name="material_silver" />
     </visual>
     <collision>
@@ -41,5 +41,5 @@
         <mesh filename="package://jetduinobot_description/meshes/battery_large/battery_large.dae"/>
       </geometry>
-      <material name="black" />
+      <xacro:insert_block name="material_black" />
     </visual>
     <collision>
@@ -72,5 +72,5 @@
         <mesh filename="package://jetduinobot_description/meshes/wheel/wheel.dae" scale="0.1 0.1 0.1"/>
       </geometry>
-      <material name="black" />
+      <xacro:insert_block name="material_black" />
     </visual>
     <collision>
@@ -98,5 +98,5 @@
         <mesh filename="package://jetduinobot_description/meshes/wheel/wheel.dae" scale="0.1 0.1 0.1"/>
       </geometry>
-      <material name="black" />
+      <xacro:insert_block name="material_black" />
     </visual>
     <collision>
@@ -125,5 +125,5 @@
         <mesh filename="package://jetduinobot_description/meshes/wheel/wheel.dae" scale="0.1 0.1 0.1"/>
       </geometry>
-      <material name="black" />
+      <xacro:insert_block name="material_black" />
     </visual>
     <collision>
@@ -151,5 +151,5 @@
         <mesh filename="package://jetduinobot_description/meshes/wheel/wheel.dae" scale="0.1 0.1 0.1"/>
       </geometry>
-      <material name="black" />
+      <xacro:insert_block name="material_black" />
     </visual>
     <collision>

Commit message: 1. Added more descriptions on how to run the jetduinobot sim 2. Added a joystick test script for driving the jetduinobot 3. Added a minimal sim launch script 4. Fixed a bug in the wheel definitions. The wheels were reversed to get them to look right, but it no longer drove correctly. I had to rotate the mesh instead.

File: jetduinobot_description/urdf/dfrobot_4wd.urdf.xacro (robot description, xacro)
@@ -96,6 +96,7 @@
     <visual>
       <geometry>
-        <mesh filename="package://jetduinobot_description/meshes/wheel/wheel.dae" scale="0.1 0.1 0.1"/>
+        <mesh filename="package://jetduinobot_description/meshes/wheel/wheel.dae" scale="0.1 0.1 0.1" />
       </geometry>
+      <origin rpy="0 3.14159 0" xyz="0 0 0"/>
       <xacro:insert_block name="material_black" />
     </visual>
@@ -116,5 +117,5 @@
     <parent link="base_link"/>
     <child link="left_rear_wheel_link"/>
-    <origin rpy="0 1.5708 0" xyz="0.07 -0.0875 -0.017"/>
+    <origin rpy="0 -1.5708 0" xyz="0.07 -0.0875 -0.017"/>
   </joint>
   <!-- front wheels -->
@@ -151,4 +152,5 @@
         <mesh filename="package://jetduinobot_description/meshes/wheel/wheel.dae" scale="0.1 0.1 0.1"/>
       </geometry>
+      <origin rpy="0 3.14159 0" xyz="0 0 0"/>
       <xacro:insert_block name="material_black" />
     </visual>
@@ -169,7 +171,11 @@
     <parent link="base_link"/>
     <child link="left_front_wheel_link"/>
-    <origin rpy="0 1.5708 0" xyz="0.07 0.0455 -0.017"/>
+    <origin rpy="0 -1.5708 0" xyz="0.07 0.0455 -0.017"/>
   </joint>
   <gazebo>
+    <plugin name="joint_state_publisher" filename="libgazebo_ros_joint_state_publisher.so">
+      <jointName>right_rear_wheel_joint, left_rear_wheel_joint, right_front_wheel_joint,
+                 left_front_wheel_joint</jointName>
+    </plugin>
     <plugin name="skid_steer_drive_controller" filename="libgazebo_ros_skid_steer_drive.so">
       <leftFrontJoint>left_front_wheel_joint</leftFrontJoint>
